File: pcb/test_linear_1/coil_driver/coil_driver/coil_driver.kicad_pcb (KiCad board)
At the start: 4 copper layers, 52 parts, among them J1 Conn_01x04_Pin, J10 Conn_01x01_Pin, J11 Conn_01x01_Pin, J12 Conn_01x01_Pin, J13 Conn_01x03_Pin, J14 Conn_01x03_Pin, J2 Conn_01x04_Pin, J3 Conn_01x04_Pin, J4 Conn_01x04_Pin, J5 Conn_01x04_Pin, J6 Conn_01x04_Pin, J7 Conn_01x04_Pin, J8 Conn_01x04_Pin, J9 Conn_01x01_Pin, Q1 BUK6D120, Q2 BUK6D120, Q3 BUK6D120, Q4 BUK6D120, Q5 BUK6D120, Q6 BUK6D120, U2 Pico

Commit message: Began PCB
Parts:
- moved C6 163.2 mm to (237.0, 74.2), turned to 90 degrees
- moved D18 162.6 mm to (232.2, 75.0), turned to 180 degrees
- moved R18 159.8 mm to (227.6, 75.0), turned to -90 degrees
- moved Q6 157.7 mm to (232.8, 69.9)
- moved R16 157.0 mm to (225.2, 75.0), turned to -90 degrees
- moved D16 152.6 mm to (225.2, 70.4), turned to 90 degrees
- moved C2 103.7 mm to (163.6, 77.4), turned to 90 degrees
- moved D6 103.0 mm to (158.8, 78.3), turned to 180 degrees
- moved D15 101.5 mm to (212.3, 75.7), turned to 180 degrees
- moved R5 100.4 mm to (154.2, 78.3), turned to -90 degrees
- moved C5 99.8 mm to (217.1, 75.0), turned to 90 degrees
- moved R3 97.6 mm to (151.9, 78.3), turned to -90 degrees
- moved Q2 97.6 mm to (158.8, 73.6)
- moved R15 95.4 mm to (207.8, 75.7), turned to -90 degrees
- moved R13 94.4 mm to (205.3, 75.7), turned to -90 degrees
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Connections:
- Q1 pad 2: /A_IN -> /coil_driver/IN2
- Q1 pad 3: GND -> /A_IN
- Q1 pad 4: (no net) -> GND
- Q1 pad 5: (no net) -> /coil_driver/IN2
- Q1 pad 6: (no net) -> /coil_driver/IN2
- Q1 pad 7: (no net) -> /coil_driver/IN2
- Q1 pad 8: (no net) -> GND
- Q2 pad 2: /B_IN -> /coil_driver1/IN2
- Q2 pad 3: GND -> /B_IN
- Q2 pad 4: (no net) -> GND
- Q2 pad 5: (no net) -> /coil_driver1/IN2
- Q2 pad 6: (no net) -> /coil_driver1/IN2
- Q2 pad 7: (no net) -> /coil_driver1/IN2
- Q2 pad 8: (no net) -> GND
- Q3 pad 2: /C_IN -> /coil_driver2/IN2
- Q3 pad 3: GND -> /C_IN
- Q3 pad 4: (no net) -> GND
- Q3 pad 5: (no net) -> /coil_driver2/IN2
- Q3 pad 6: (no net) -> /coil_driver2/IN2
- Q3 pad 7: (no net) -> /coil_driver2/IN2
- Q3 pad 8: (no net) -> GND
- Q4 pad 2: /D_IN -> /coil_driver3/IN2
- Q4 pad 3: GND -> /D_IN
- Q4 pad 4: (no net) -> GND
- Q4 pad 5: (no net) -> /coil_driver3/IN2
- Q4 pad 6: (no net) -> /coil_driver3/IN2
- Q4 pad 7: (no net) -> /coil_driver3/IN2
- Q4 pad 8: (no net) -> GND
- Q5 pad 2: /E_IN -> /coil_driver4/IN2
- Q5 pad 3: GND -> /E_IN
- Q5 pad 4: (no net) -> GND
- Q5 pad 5: (no net) -> /coil_driver4/IN2
- Q5 pad 6: (no net) -> /coil_driver4/IN2
- Q5 pad 7: (no net) -> /coil_driver4/IN2
- Q5 pad 8: (no net) -> GND
- Q6 pad 2: /F_IN -> /coil_driver5/IN2
- Q6 pad 3: GND -> /F_IN
- Q6 pad 4: (no net) -> GND
- Q6 pad 5: (no net) -> /coil_driver5/IN2
- Q6 pad 6: (no net) -> /coil_driver5/IN2
- Q6 pad 7: (no net) -> /coil_driver5/IN2
- Q6 pad 8: (no net) -> GND
Routing:
- net GND: track 0.00 -> 46.2 mm
- net VCC: track 0.00 -> 17.1 mm
- net /coil_driver/IN2: track 0.00 -> 13.0 mm, vias 0 -> 2
- net /coil_driver5/IN2: track 0.00 -> 11.6 mm, vias 0 -> 2
- net /F_IN: track 0.00 -> 10.7 mm
- net /coil_driver4/IN2: track 0.00 -> 10.5 mm, vias 0 -> 2
- net /E_IN: track 0.00 -> 10.2 mm
- net /B_IN: track 0.00 -> 10.1 mm
- net /C_IN: track 0.00 -> 10.1 mm
- net /A_IN: track 0.00 -> 9.95 mm
- net /D_IN: track 0.00 -> 9.34 mm
- net /coil_driver1/IN2: track 0.00 -> 8.66 mm, vias 0 -> 2
- net /coil_driver3/IN2: track 0.00 -> 8.64 mm, vias 0 -> 2
- net /coil_driver2/IN2: track 0.00 -> 8.34 mm, vias 0 -> 2
- net Net-(D7-K): track 0.00 -> 1.94 mm
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