File: pcb/coil_driver/coil_module1.kicad_sch (KiCad schematic)
At the start: 0 parts

Commit message: Almost finished PCB
Parts:
- added TP1, TP11, TP12, TP13, TP14, TP2, TP3, TP4: TestPoint_2Pole, pads:pad_dual, symbol Connector:TestPoint_2Pole
Connections:
- net A1: now also TP11.1
- new net B1: TP12.1
- new net C1: TP4.1
- new net COIL_A1: TP1.2, TP11.2
- new net COIL_B1: TP12.2, TP2.2
- new net COIL_C1: TP3.2, TP4.2
- new net COIL_D1: TP13.2, TP14.2
- new net D1: TP13.1
- new net PWR: TP1.1, TP14.1, TP2.1, TP3.1
