File: pcb/coil_driver/coil_module2.kicad_sch (KiCad schematic)
At the start: 0 parts

Commit message: Almost finished PCB
Parts:
- added TP10, TP15, TP16, TP17, TP18, TP19, TP20, TP5, TP6, TP7, TP8, TP9: TestPoint_2Pole, pads:pad_dual, symbol Connector:TestPoint_2Pole
Connections:
- net A2: now also TP15.1
- new net B2: TP16.1
- new net C2: TP18.1
- new net COIL_A2: TP15.2, TP5.2
- new net COIL_B2: TP16.2, TP6.2
- new net COIL_C2: TP17.2, TP18.2
- new net COIL_D2: TP7.2, TP8.2
- new net COIL_E2: TP10.2, TP9.2
- new net COIL_F2: TP19.2, TP20.2
- new net D2: TP7.1
- new net E2: TP9.1
- new net F2: TP19.1
- new net PWR: TP10.1, TP17.1, TP20.1, TP5.1, TP6.1, TP8.1
