File: pcb/coil_driver/coil_driver.kicad_pcb (KiCad board)
At the start: 4 copper layers, 52 parts, among them J1 Conn_01x04_Pin, J10 Conn_01x01_Pin, J11 Conn_01x01_Pin, J12 Conn_01x01_Pin, J13 Conn_01x03_Pin, J14 Conn_01x03_Pin, J2 Conn_01x04_Pin, J3 Conn_01x04_Pin, J4 Conn_01x04_Pin, J5 Conn_01x04_Pin, J6 Conn_01x04_Pin, J7 Conn_01x04_Pin, J8 Conn_01x04_Pin, J9 Conn_01x01_Pin, Q1 BUK6D120, Q2 BUK6D120, Q3 BUK6D120, Q4 BUK6D120, Q5 BUK6D120, Q6 BUK6D120, U2 Pico

Commit message: Almost finished PCB
Parts:
- added L1: rounded_coil, PCB Coils:rounded_thin, F.Cu at (47.0, 32.0)
- added L10: rounded_coil, PCB Coils:rounded_thicc, F.Cu at (163.0, 32.0)
- added L11: rounded_coil, PCB Coils:rounded_thicc, F.Cu at (142.0, 32.0)
- added L12: rounded_coil, PCB Coils:rounded_thicc, F.Cu at (121.0, 31.5)
- added L2: rounded_coil, PCB Coils:rounded_thin, F.Cu at (68.0, 32.0)
- added L3: rounded_coil, PCB Coils:rounded_thin, F.Cu at (89.0, 32.0)
- added L4: rounded_coil, PCB Coils:rounded_thin, F.Cu at (89.0, 52.5)
- added L5: rounded_coil, PCB Coils:rounded_thin, F.Cu at (68.0, 52.5)
- added L6: rounded_coil, PCB Coils:rounded_thin, F.Cu at (47.0, 52.5)
- added L7: rounded_coil, PCB Coils:rounded_thicc, F.Cu at (121.0, 51.5)
- added L8: rounded_coil, PCB Coils:rounded_thicc, F.Cu at (142.0, 52.0)
- added L9: rounded_coil, PCB Coils:rounded_thicc, F.Cu at (163.0, 52.0)
- added TP1: TestPoint_2Pole, pads:pad_dual, F.Cu at (34.5, 71.1)
- added TP10: TestPoint_2Pole, pads:pad_dual, F.Cu at (164.3, 170.8)
- added TP11: TestPoint_2Pole, pads:pad_dual, F.Cu at (86.2, 146.3)
- added TP12: TestPoint_2Pole, pads:pad_dual, F.Cu at (98.4, 146.3)
- added TP13: TestPoint_2Pole, pads:pad_dual, F.Cu at (123.6, 146.3)
- added TP14: TestPoint_2Pole, pads:pad_dual, F.Cu at (32.8, 66.8)
- added TP15: TestPoint_2Pole, pads:pad_dual, F.Cu at (88.8, 146.3)
- added TP16: TestPoint_2Pole, pads:pad_dual, F.Cu at (101.0, 146.3)
- added TP17: TestPoint_2Pole, pads:pad_dual, F.Cu at (105.2, 129.8)
- added TP18: TestPoint_2Pole, pads:pad_dual, F.Cu at (113.4, 146.3)
- added TP19: TestPoint_2Pole, pads:pad_dual, F.Cu at (140.8, 146.3)
- added TP2: TestPoint_2Pole, pads:pad_dual, F.Cu at (34.5, 71.9)
- added TP20: TestPoint_2Pole, pads:pad_dual, F.Cu at (174.5, 64.3)
- added TP3: TestPoint_2Pole, pads:pad_dual, F.Cu at (33.3, 67.8)
- added TP4: TestPoint_2Pole, pads:pad_dual, F.Cu at (110.9, 146.3)
- added TP5: TestPoint_2Pole, pads:pad_dual, F.Cu at (170.2, 140.6)
- added TP6: TestPoint_2Pole, pads:pad_dual, F.Cu at (180.3, 130.6)
- added TP7: TestPoint_2Pole, pads:pad_dual, F.Cu at (126.1, 146.3)
- added TP8: TestPoint_2Pole, pads:pad_dual, F.Cu at (171.7, 140.6)
- added TP9: TestPoint_2Pole, pads:pad_dual, F.Cu at (136.0, 146.3)
- moved J1 0.22 mm to (86.2, 152.8)
- moved J2 0.22 mm to (86.2, 150.2)
- moved J4 0.05 mm to (98.4, 150.2)
- moved J3 0.05 mm to (98.4, 152.8)
- moved J5 0.05 mm to (110.9, 152.8)
- moved J6 0.05 mm to (110.9, 150.2)
- moved J8 0.05 mm to (123.6, 150.2)
- moved J7 0.05 mm to (123.6, 152.8)
Connections:
- J11 pad 1: VCC -> /E2
- J12 pad 1: VCC -> /F2
- J2 pad 1: VCC -> /A1
- J2 pad 2: VCC -> /A2
- J2 pad 3: VCC -> /A3
- J2 pad 4: VCC -> /A4
- J4 pad 1: VCC -> /B1
- J4 pad 2: VCC -> /B2
- J4 pad 3: VCC -> /B3
- J4 pad 4: VCC -> /B4
- J6 pad 1: VCC -> /C1
- J6 pad 2: VCC -> /C2
- J6 pad 3: VCC -> /C3
- J6 pad 4: VCC -> /C4
- J8 pad 1: VCC -> /D1
- J8 pad 2: VCC -> /D2
- J8 pad 3: VCC -> /D3
- J8 pad 4: VCC -> /D4
Routing:
- net /coil_module2/COIL_A2: track 0.00 -> 3365.4 mm, vias 0 -> 51
- net /coil_module1/COIL_A1: track 0.00 -> 2417.2 mm, vias 0 -> 38
- net /coil_module1/COIL_B1: track 0.00 -> 2402.8 mm, vias 0 -> 40
- net /coil_module1/COIL_D1: track 0.00 -> 2358.9 mm, vias 0 -> 38
- net /coil_module1/COIL_C1: track 0.00 -> 2344.3 mm, vias 0 -> 38
- net /coil_module2/COIL_B2: track 0.00 -> 1716.8 mm, vias 0 -> 26
- net /coil_module2/COIL_D2: track 0.00 -> 1705.0 mm, vias 0 -> 50
- net /coil_module2/COIL_C2: track 0.00 -> 1672.7 mm, vias 0 -> 26
- net /coil_module2/COIL_F2: track 0.00 -> 1672.5 mm, vias 0 -> 25
- net /B1: track 0.00 -> 2.74 mm
- net /coil_module2/COIL_E2: vias 0 -> 24

Commit message: PCB Should be finished
Parts:
- J10, J11, J12, J9: value Conn_01x01_Pin -> Conn_01x04_Pin; footprint Connector_PinHeader_2.54mm:PinHeader_1x01_P2.54mm_Vertical -> Connector_PinHeader_2.54mm:PinHeader_1x04_P2.54mm_Vertical
- moved TP10 142.8 mm to (280.8, 88.2), turned to 180 degrees
- moved J11 122.1 mm to (254.9, 178.3)
- moved TP8 120.8 mm to (280.9, 89.0), turned to 180 degrees
- moved TP19 119.3 mm to (257.4, 171.8)
- moved J12 116.8 mm to (254.9, 175.7)
- moved TP9 111.9 mm to (245.0, 171.8)
- moved TP17 111.3 mm to (211.9, 98.2)
- moved TP14 110.6 mm to (140.4, 92.3)
- moved TP3 110.1 mm to (140.4, 93.3)
- moved Q6 109.6 mm to (233.4, 206.7)
- moved J9 109.4 mm to (242.4, 178.3)
- moved D7 109.4 mm to (226.0, 188.6)
- moved TP20 109.4 mm to (280.9, 89.7)
- moved C2 109.4 mm to (222.8, 192.5)
- moved C4 109.4 mm to (207.2, 210.3)
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Connections:
- J10 pad 1: /F_OUT -> /E1
- J11 pad 1: /E2 -> /F_OUT
- J12 pad 1: /F2 -> /F1
- L11 pad 2: /coil_module3/E3 -> /E3
- L12 pad 2: /coil_module3/F3 -> /F3
- L5 pad 2: /coil_module4/E4 -> /E4
- L6 pad 2: /coil_module4/F4 -> /F4
Routing:
- net /coil_module2/COIL_E2: track 0.00 -> 1696.6 mm, vias 24 -> 26
- net /coil_module2/COIL_A2: track 3365.4 -> 1671.1 mm, vias 51 -> 50
- net /E4: track 0.00 -> 344.7 mm, vias 0 -> 1
- net /F4: track 0.00 -> 308.5 mm, vias 0 -> 1
- net /C4: track 0.00 -> 285.5 mm, vias 0 -> 1
- net /F3: track 0.00 -> 222.0 mm, vias 0 -> 1
- net /E3: track 0.00 -> 208.6 mm, vias 0 -> 1
- net /A4: track 0.00 -> 203.4 mm, vias 0 -> 1
- net /D3: track 0.00 -> 194.9 mm, vias 0 -> 1
- net /B4: track 0.00 -> 172.3 mm, vias 0 -> 2
- net /C3: track 0.00 -> 157.2 mm
- net /D4: track 0.00 -> 133.9 mm, vias 0 -> 5
- net /B3: track 0.00 -> 121.8 mm
- net /A3: track 0.00 -> 109.5 mm, vias 0 -> 1
- net VCC: track 17.1 -> 100.1 mm, vias 0 -> 17
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- added copper zone on F.Cu, net GND
- added copper zone on In1.Cu, net GND
- added copper zone on In2.Cu, net GND
- added copper zone on B.Cu, net VCC
Other:
- board outline added: 168 x 187 mm
- board text added: "1-2-3-4"
- board text added: "A"
- board text added: "B"
- board text added: "C"
- board text added: "D"
- board text added: "E"
- board text added: "F"
- board text added: "GND"
- board text added: "MODULE 1"
- board text added: "MODULE 2"
- board text added: "MODULE 3"
- board text added: "MODULE 4"
- board text added: "VCC"

Commit message: Finished PCB
Parts:
- moved L7 0.51 mm to (227.3, 77.5)
Other:
- board text added: "COIL TESTER V0.1 Jonas Stirnemann BACHELOR 2024"
- board text added: "MODULE 1 : - 2 coils / layer - 20 mils traces - 10 mils gap"
- board text added: "MODULE 2 : - 3 coils / layer - 20 mils traces - 10 mils gap"
- board text added: "MODULE 3 : - 2 layers - 10 mils width - 5 mils gap - 25 coils per layer"
- board text added: "MODULE 4 : - 2 layers - 3.5 mils width - 3.5 mils gap - 50 coils per layer"
