File: pcb/coil_driver/coil_driver.kicad_sch (KiCad schematic)
At the start: 16 parts, among them J1 Conn_01x04_Pin, J10 Conn_01x01_Pin, J11 Conn_01x01_Pin, J12 Conn_01x01_Pin, J13 Conn_01x03_Pin, J14 Conn_01x03_Pin, J2 Conn_01x04_Pin, J3 Conn_01x04_Pin, J4 Conn_01x04_Pin, J5 Conn_01x04_Pin, J6 Conn_01x04_Pin, J7 Conn_01x04_Pin, J8 Conn_01x04_Pin, J9 Conn_01x01_Pin, U2 Pico

Commit message: PCB Should be finished
Parts:
- removed J10, J11, J12, J9: Conn_01x01_Pin, Connector_PinHeader_2.54mm:PinHeader_1x01_P2.54mm_Vertical, symbol Connector:Conn_01x01_Pin
- added J10, J11, J12, J9: Conn_01x04_Pin, Connector_PinHeader_2.54mm:PinHeader_1x04_P2.54mm_Vertical, symbol Connector:Conn_01x04_Pin
Connections:
- net E2: now also J10.2 (Pin_2)
- net E_OUT: now also J9.1 (Pin_1), J9.2 (Pin_2), J9.3 (Pin_3), J9.4 (Pin_4)
- net F2: now also J12.2 (Pin_2)
- net F_OUT: now also J11.1 (Pin_1), J11.2 (Pin_2), J11.3 (Pin_3), J11.4 (Pin_4)
- new net E1: J10.1 (Pin_1)
- new net E3: J10.3 (Pin_3)
- new net E4: J10.4 (Pin_4)
- new net F1: J12.1 (Pin_1)
- new net F3: J12.3 (Pin_3)
- new net F4: J12.4 (Pin_4)
Other:
- sheet coil_module3 ports: added E3, F3; removed none
- sheet coil_module4 ports: added E4, F4; removed none

Commit message: Fixed tictactoe
Parts:
- J1, J10, J11, J12, J13, J14, J2, J3, J4, J5, J6, J7, J8, J9: MFR (none) -> 826629-4; MOUSER (none) -> 571-826629-4
- U2: MFR (none) -> SC0915; MOUSER (none) -> 358-SC0915
