File: pcb/coil_driver/single_coil.kicad_sch (KiCad schematic)
At the start: 6 parts, among them Q1 BUK6D120

Commit message: Almost finished PCB
Parts:
- renumbered C1 to C2, D1 to D2, D4 to D6, Q1 to Q2, R1 to R3, R2 to R5
Changed lines of the file:
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@@
 		(on_board yes)
 		(dnp no)
-		(property "Reference" "R2"
+		(property "Reference" "R5"
 			(at 100.076 67.564 0)
 			(effects
@@
 		(on_board yes)
 		(dnp no)
-		(property "Reference" "Q1"
+		(property "Reference" "Q2"
 			(at 109.982 60.198 0)
 			(effects
@@
 		(on_board yes)
 		(dnp no)
-		(property "Reference" "#PWR01"
+		(property "Reference" "#PWR06"
 			(at 83.82 82.55 0)
 			(effects
@@
 		(on_board yes)
 		(dnp no)
-		(property "Reference" "#PWR04"
+		(property "Reference" "#PWR09"
 			(at 107.95 40.64 0)
 			(effects
@@
 		(on_board yes)
 		(dnp no)
-		(property "Reference" "#PWR013"
+		(property "Reference" "#PWR015"
 			(at 83.82 60.96 0)
 			(effects
@@
 		(on_board yes)
 		(dnp no)
-		(property "Reference" "R1"
+		(property "Reference" "R3"
 			(at 85.09 71.12 0)
 			(effects
@@
 		(on_board yes)
 		(dnp no)
-		(property "Reference" "D4"
+		(property "Reference" "D6"
 			(at 112.268 52.07 0)
 			(effects
@@
 		(on_board yes)
 		(dnp no)
-		(property "Reference" "#PWR02"
+		(property "Reference" "#PWR03"
 			(at 107.95 82.55 0)
 			(effects
@@
 		(on_board yes)
 		(dnp no)
-		(property "Reference" "#PWR032"
+		(property "Reference" "#PWR033"
 			(at 83.82 40.64 0)
 			(effects
@@
 		(on_board yes)
 		(dnp no)
-		(property "Reference" "D1"
+		(property "Reference" "D2"
 			(at 85.344 66.04 90)
 			(effects
@@
 		(dnp no)
 		(fields_autoplaced yes)
-		(property "Reference" "C1"
+		(property "Reference" "C2"
 			(at 86.36 44.4562 0)
 			(effects

Commit message: Fixed tictactoe
Parts:
- R3: MFR (none) -> ERJ-S08F1001V; MOUSER (none) -> 667-ERJ-S08F1001V
- R5: MFR (none) -> RCV1206120KFKEA; MOUSER (none) -> 71-RCV1206120KFKEA
Changed lines of the file:
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@@
+			)
+		)
+		(property "MFR" "RCV1206120KFKEA "
+			(at 99.06 68.58 0)
+			(effects
+				(font
+					(size 1.27 1.27)
+				)
+				(hide yes)
+			)
+		)
+		(property "MOUSER" " 71-RCV1206120KFKEA "
+			(at 99.06 68.58 0)
+			(effects
+				(font
+					(size 1.27 1.27)
+				)
+				(hide yes)
 			)
 		)
@@
 			(at 83.82 72.39 0)
 			(effects
+				(font
+					(size 1.27 1.27)
+				)
+				(hide yes)
+			)
+		)
+		(property "MFR" " ERJ-S08F1001V "
+			(at 83.82 72.39 0)
+			(effects
+				(font
+					(size 1.27 1.27)
+				)
+				(hide yes)
+			)
+		)
+		(property "MOUSER" " 667-ERJ-S08F1001V "
+			(at 83.82 72.39 0)
+			(effects
