File: pcb/only_coils/sub_coils/sub_coils.kicad_sch (KiCad schematic)
At the start: 8 parts, among them J2 Conn_01x06_Pin, J4 Conn_01x03_Pin

Commit message: Added small script for square coils
Parts:
- L1, L3, L4: footprint sub_coils:sub_coil -> sub_coils:sub_coil_small_2
Changed lines of the file:
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@@
 			)
 		)
-		(property "Footprint" "sub_coils:sub_coil"
+		(property "Footprint" "sub_coils:sub_coil_small_2"
 			(at 113.665 73.66 90)
 			(effects
@@
 			)
 		)
-		(property "Footprint" "sub_coils:sub_coil"
+		(property "Footprint" "sub_coils:sub_coil_small_2"
 			(at 164.465 73.66 90)
 			(effects
@@
 			)
 		)
-		(property "Footprint" "sub_coils:sub_coil"
+		(property "Footprint" "sub_coils:sub_coil_small_2"
 			(at 126.365 55.88 90)
 			(effects
